File: USBTinyISP-Single-Sided/usbtinyisp v2.0 SS.brd (EAGLE design)
At the start: 68.2 x 36.8 mm, 24 parts, among them IC1 ATTINY2313-20P, IC2 74AHC125N, Q1 12Mhz

Commit message: Version 0.01
Parts:
- removed JP4: BUS, pinhead:1X02
- removed JP5: PGM, pinhead:1X02
- moved C2 5.08 mm to (16.5, 33.0)
Connections:
- net N$9: no longer JP5.1
- net RST: no longer JP5.2
- net VCC: no longer JP4.1, JP4.2
Routing:
- net RST: track 51.9 -> 27.7 mm, vias 2 -> 0
- net N$9: track 13.5 -> 4.34 mm
- net GND: track 196.4 -> 201.5 mm
- net VCC: track 69.1 -> 67.7 mm
