File: USBTinyISP-Single-Sided/usbtiny-v2-SS.brd (EAGLE design)
At the start: 68.2 x 36.8 mm, 22 parts, among them IC1 ATTINY2313-20P, IC2 74AHC125N, Q1 12Mhz

Commit message: Version 0.03
Parts:
- R3, R6: device rcl-ez:0207/5V -> rcl-ez:0207/10
- moved R3 27.2 mm to (15.2, 20.3), turned to 270 degrees
- moved C1 23.6 mm to (21.6, 33.0), turned to 270 degrees
- moved R6 9.25 mm to (58.4, 10.2), turned to 180 degrees
- moved LED1 4.58 mm to (49.5, 10.2)
- moved D2 2.54 mm to (12.7, 20.3)
- moved D1 2.54 mm to (10.2, 20.3)
- moved R1 1.27 mm to (17.8, 20.3)
- moved R2 1.27 mm to (20.3, 21.6)
Routing:
- net GND: track 201.5 -> 127.6 mm
- net N$1: track 77.3 -> 12.8 mm, vias 2 -> 0
- net N$16: track 5.08 -> 28.6 mm
- net RST: track 27.7 -> 16.8 mm
- net N$2: track 28.2 -> 19.8 mm
- net VCC: track 67.7 -> 73.9 mm, vias 2 -> 0
- net N$6: track 11.4 -> 12.7 mm
- net N$3: track 14.0 -> 15.2 mm
- net N$7: track 6.35 -> 7.62 mm
- net N$8: track 3.59 -> 2.54 mm
