File: USBTinyISP-Single-Sided/usbtiny-v2-SS.brd (EAGLE design)
At the start: 68.2 x 36.8 mm, 22 parts, among them IC1 ATTINY2313-20P, IC2 74AHC125N, Q1 12Mhz

Commit message: Version 0.02
Parts:
- R7: device rcl-ez:0204/5 -> rcl-ez:0207/10
- moved R7 11.4 mm to (58.4, 22.9), turned to 90 degrees
Connections:
- net N$15 renamed BUFFEN
Routing:
- net BUFFEN: track 49.9 -> 64.7 mm, vias 2 -> 0
- net SCK: track 17.8 -> 5.61 mm, vias 2 -> 0
- net N$12: track 16.5 -> 11.2 mm, vias 2 -> 0
Changed lines of the file:
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@@
 <attribute name="VALUE" x="12.7" y="22.606" size="1.27" layer="27" ratio="10" rot="R270"/>
 </element>
-<element name="R7" library="rcl-ez" package="0204/5" value="1.5K" x="58.42" y="34.29" smashed="yes" rot="R180">
-<attribute name="NAME" x="61.6966" y="33.1216" size="0.9906" layer="25" ratio="12" rot="R180"/>
-<attribute name="VALUE" x="60.5536" y="36.6014" size="0.9906" layer="27" ratio="12" rot="R180"/>
+<element name="R7" library="rcl-ez" package="0207/10" value="1.5K" x="58.42" y="22.86" smashed="yes" rot="R90">
+<attribute name="NAME" x="59.1566" y="16.6116" size="0.9906" layer="25" ratio="12" rot="R180"/>
+<attribute name="VALUE" x="60.7314" y="20.7264" size="0.9906" layer="27" ratio="12" rot="R90"/>
 </element>
 <element name="R4" library="rcl-ez" package="0207/10" value="1.5K" x="60.96" y="12.7" rot="R180"/>
@@
 <wire x1="8.89" y1="20.32" x2="10.16" y2="20.32" width="1.016" layer="16"/>
 <wire x1="10.16" y1="20.32" x2="10.16" y2="31.75" width="1.016" layer="1"/>
-<wire x1="24.13" y1="34.29" x2="29.21" y2="29.21" width="0.6096" layer="16"/>
-<wire x1="29.21" y1="29.21" x2="39.37" y2="29.21" width="0.6096" layer="16"/>
-<wire x1="39.37" y1="29.21" x2="40.64" y2="30.48" width="0.6096" layer="16"/>
 <wire x1="45.72" y1="33.02" x2="45.72" y2="34.29" width="1.016" layer="16"/>
 <wire x1="43.18" y1="30.48" x2="45.72" y2="33.02" width="1.016" layer="16"/>
@@
 <wire x1="16.51" y1="34.29" x2="24.13" y2="34.29" width="1.016" layer="16"/>
 <wire x1="7.25" y1="21.61" x2="7.6" y2="21.61" width="1.016" layer="16"/>
+<wire x1="40.64" y1="30.48" x2="36.83" y2="30.48" width="0.6096" layer="16"/>
+<wire x1="36.83" y1="30.48" x2="35.56" y2="29.21" width="0.6096" layer="16"/>
+<wire x1="35.56" y1="29.21" x2="29.21" y2="29.21" width="0.6096" layer="16"/>
+<wire x1="29.21" y1="29.21" x2="24.13" y2="34.29" width="0.6096" layer="16"/>
 </signal>
 <signal name="GND">
@@
 <contactref element="R7" pad="1"/>
 <contactref element="JP1" pad="3"/>
-<wire x1="58.42" y1="21.59" x2="60.96" y2="21.59" width="1.016" layer="16"/>
-<wire x1="58.42" y1="21.59" x2="58.42" y2="33.02" width="1.016" layer="1"/>
-<wire x1="60.96" y1="33.02" x2="60.96" y2="34.29" width="1.016" layer="16"/>
-<wire x1="58.42" y1="33.02" x2="60.96" y2="33.02" width="1.016" layer="16"/>
-<via x="58.42" y="21.59" extent="1-16" drill="0.9" diameter="1.778"/>
-<via x="58.42" y="33.02" extent="1-16" drill="0.9" diameter="1.778"/>
+<wire x1="60.96" y1="21.59" x2="59.69" y2="21.59" width="1.016" layer="16"/>
+<wire x1="59.69" y1="21.59" x2="58.42" y2="20.32" width="1.016" layer="16"/>
+<wire x1="58.42" y1="20.32" x2="58.42" y2="17.78" width="1.016" layer="16"/>
 </signal>
 <signal name="RST">
@@
 <contactref element="R7" pad="2"/>
 <contactref element="IC2" pad="3"/>
-<wire x1="53.34" y1="34.29" x2="55.88" y2="34.29" width="1.016" layer="16"/>
-<wire x1="53.34" y1="25.4" x2="53.34" y2="34.29" width="1.016" layer="1"/>
-<wire x1="48.26" y1="25.4" x2="53.34" y2="25.4" width="0.6096" layer="16"/>
-<via x="53.34" y="34.29" extent="1-16" drill="0.9" diameter="1.778"/>
-<via x="53.34" y="25.4" extent="1-16" drill="0.9" diameter="1.778"/>
+<wire x1="48.26" y1="25.4" x2="50.8" y2="25.4" width="0.6096" layer="16"/>
+<wire x1="50.8" y1="25.4" x2="52.07" y2="26.67" width="0.6096" layer="16"/>
+<wire x1="52.07" y1="26.67" x2="57.15" y2="26.67" width="0.6096" layer="16"/>
+<wire x1="57.15" y1="26.67" x2="58.42" y2="27.94" width="0.6096" layer="16"/>
 </signal>
 <signal name="N$13">
@@
 <wire x1="41.91" y1="21.59" x2="40.64" y2="22.86" width="0.6096" layer="16"/>
 </signal>
-<signal name="N$15">
+<signal name="BUFFEN">
 <contactref element="IC1" pad="8"/>
 <contactref element="IC2" pad="10"/>
@@
 <contactref element="IC2" pad="1"/>
 <contactref element="IC2" pad="13"/>
-<wire x1="55.88" y1="20.32" x2="54.61" y2="20.32" width="0.254" layer="16"/>
-<wire x1="49.53" y1="30.48" x2="48.26" y2="30.48" width="1.016" layer="16"/>
-<wire x1="50.8" y1="29.21" x2="49.53" y2="30.48" width="1.016" layer="16"/>
-<wire x1="50.8" y1="29.21" x2="53.34" y2="29.21" width="1.016" layer="16"/>
-<wire x1="53.34" y1="29.21" x2="54.61" y2="27.94" width="1.016" layer="16"/>
-<wire x1="54.61" y1="27.94" x2="55.88" y2="27.94" width="1.016" layer="16"/>
-<wire x1="48.26" y1="22.86" x2="50.8" y2="22.86" width="0.6096" layer="16"/>
-<wire x1="50.8" y1="22.86" x2="50.8" y2="29.21" width="1.016" layer="1"/>
-<wire x1="50.8" y1="22.86" x2="53.34" y2="20.32" width="0.6096" layer="16"/>
-<wire x1="53.34" y1="20.32" x2="55.88" y2="20.32" width="0.6096" layer="16"/>
 <wire x1="44.45" y1="22.86" x2="48.26" y2="22.86" width="0.6096" layer="16"/>
 <wire x1="43.18" y1="24.13" x2="44.45" y2="22.86" width="0.6096" layer="16"/>
@@
 <wire x1="34.29" y1="12.7" x2="36.83" y2="15.24" width="0.6096" layer="16"/>
 <wire x1="33.02" y1="12.7" x2="34.29" y2="12.7" width="0.6096" layer="16"/>
-<via x="50.8" y="29.21" extent="1-16" drill="0.9" diameter="1.778"/>
-<via x="50.8" y="22.86" extent="1-16" drill="0.7" diameter="1.27"/>
+<wire x1="48.26" y1="22.86" x2="50.8" y2="22.86" width="0.6096" layer="16"/>
+<wire x1="50.8" y1="22.86" x2="53.34" y2="20.32" width="0.6096" layer="16"/>
+<wire x1="53.34" y1="20.32" x2="55.88" y2="20.32" width="0.6096" layer="16"/>
+<wire x1="48.26" y1="30.48" x2="50.8" y2="30.48" width="0.6096" layer="16"/>
+<wire x1="50.8" y1="30.48" x2="53.34" y2="27.94" width="0.6096" layer="16"/>
+<wire x1="53.34" y1="27.94" x2="55.88" y2="27.94" width="0.6096" layer="16"/>
+<wire x1="48.26" y1="30.48" x2="46.99" y2="30.48" width="0.6096" layer="16"/>
+<wire x1="46.99" y1="30.48" x2="45.72" y2="29.21" width="0.6096" layer="16"/>
+<wire x1="45.72" y1="29.21" x2="38.1" y2="29.21" width="0.6096" layer="16"/>
+<wire x1="38.1" y1="29.21" x2="36.83" y2="27.94" width="0.6096" layer="16"/>
+<wire x1="36.83" y1="27.94" x2="36.83" y2="25.4" width="0.6096" layer="16"/>
+<wire x1="36.83" y1="25.4" x2="36.83" y2="24.765" width="0.6096" layer="16"/>
+<wire x1="36.83" y1="24.765" x2="36.83" y2="24.13" width="0.6096" layer="16"/>
+<wire x1="36.83" y1="24.13" x2="36.83" y2="23.495" width="0.6096" layer="16"/>
+<wire x1="36.83" y1="23.495" x2="36.83" y2="22.86" width="0.6096" layer="16"/>
+<wire x1="38.1" y1="24.13" x2="36.83" y2="25.4" width="0.6096" layer="16"/>
+<wire x1="38.1" y1="24.13" x2="37.465" y2="24.13" width="0.6096" layer="16"/>
+<wire x1="37.465" y1="24.13" x2="36.83" y2="24.13" width="0.6096" layer="16"/>
+<wire x1="36.83" y1="24.765" x2="37.465" y2="24.13" width="0.6096" layer="16"/>
+<wire x1="36.83" y1="23.495" x2="37.465" y2="24.13" width="0.6096" layer="16"/>
 </signal>
 <signal name="MISO'">

Commit message: Version 0.03
Parts:
- R2: device rcl-ez:0207/7 -> rcl-ez:0207/10
- R3: device rcl-ez:0207/5V -> rcl-ez:0207/10
- R5, R6: device rcl-ez:0207/5V -> rcl-ez:0207/2V
- moved R3 14.5 mm to (25.4, 12.7)
- moved D1 12.8 mm to (11.4, 7.62), turned to 180 degrees
- moved D2 10.9 mm to (11.4, 10.2), turned to 180 degrees
- moved R1 8.13 mm to (25.4, 15.2), turned to 0 degrees
- moved R6 5.39 mm to (53.3, 11.4)
- moved R2 5.39 mm to (25.4, 17.8), turned to 0 degrees
- moved LED1 4.58 mm to (49.5, 10.2)
- moved LED2 3.81 mm to (27.9, 5.08), turned to 270 degrees
- moved R5 2.54 mm to (29.2, 10.2), turned to 0 degrees
- moved X1 1.80 mm to (3.81, 24.1)
- moved C3 0.64 mm to (25.4, 26.7)
- moved C4 0.64 mm to (25.4, 21.6)
Routing:
- net N$1: track 77.3 -> 23.4 mm, vias 2 -> 0
- net GND: track 201.5 -> 158.2 mm
- net N$20: track 40.9 -> 0.00 mm
- net N$19: track 27.9 -> 0.00 mm
- net N$5: track 25.8 -> 0.00 mm, vias 1 -> 0
- net N$4: track 19.1 -> 0.00 mm
- net N$3: track 14.0 -> 2.54 mm
- net RST: track 27.7 -> 16.8 mm
- net N$6: track 11.4 -> 2.54 mm
- net N$16: track 5.08 -> 12.3 mm
- net N$2: track 28.2 -> 33.8 mm
- net VCC: track 67.7 -> 69.4 mm
- net N$10: track 3.81 -> 2.54 mm
- net N$7: track 6.35 -> 7.62 mm
- net N$8: track 3.59 -> 2.54 mm
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Other:
- board text removed: "JQ"

Commit message: Version 0.04
Parts:
- moved JP3 17.3 mm to (63.5, 29.2), turned to 90 degrees
- moved C2 8.13 mm to (21.6, 26.7)
- moved R10 5.39 mm to (25.4, 30.5)
Routing:
- net VCC: track 69.4 -> 89.7 mm
- net N$14: track 20.2 -> 12.5 mm
- net GND: track 158.2 -> 156.1 mm
- net N$9: track 4.34 -> 2.54 mm
- net MOSI: track 11.4 -> 9.94 mm

Commit message: Version 0.05
Parts:
- moved R6 11.7 mm to (41.9, 8.89)
- moved IC2 11.7 mm to (40.6, 20.3)
- moved JP1 11.7 mm to (50.8, 19.1)
- moved JP3 11.7 mm to (52.1, 26.7)
- moved LED1 11.7 mm to (38.1, 7.62)
- moved R4 11.7 mm to (49.5, 10.2)
- moved R7 11.7 mm to (47.0, 20.3)
- moved R5 8.03 mm to (21.6, 7.62)
- moved C2 8.03 mm to (14.0, 24.1), turned to 180 degrees
- moved Q1 8.03 mm to (21.6, 21.6)
- moved C3 8.03 mm to (17.8, 24.1)
- moved C4 8.03 mm to (17.8, 19.1)
- moved IC1 8.03 mm to (29.2, 16.5)
- moved R1 8.03 mm to (17.8, 12.7)
- moved R10 8.03 mm to (17.8, 27.9)
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Routing:
- net GND: track 156.1 -> 135.3 mm
- net N$2: track 33.8 -> 24.5 mm
- net VCC: track 89.7 -> 80.7 mm
- net BUFFEN: track 64.7 -> 57.1 mm
- net MISO': track 16.3 -> 12.5 mm
- net SCK': track 7.62 -> 3.81 mm
- net RST': track 7.62 -> 3.81 mm
- net N$7: track 7.62 -> 3.81 mm
- net MOSI': track 17.3 -> 13.5 mm
- net N$14: track 12.5 -> 14.3 mm
- net N$1: track 23.4 -> 25.1 mm
- net N$11: track 3.81 -> 2.54 mm
Other:
- board size 68.2 x 36.8 mm -> 56.8 x 33 mm

Commit message: Version 0.06
Parts:
- moved JP1 3.81 mm to (50.8, 15.2)
- moved R6 2.84 mm to (40.6, 6.35), turned to 90 degrees
- moved R4 2.54 mm to (49.5, 7.62)
- moved LED1 1.27 mm to (36.8, 7.62)
Routing:
- net GND: track 135.3 -> 127.0 mm
- net N$14: track 14.3 -> 18.1 mm
- net SCK: track 5.61 -> 2.54 mm
- net MISO: track 5.61 -> 8.67 mm
- net RST: track 16.8 -> 13.8 mm
- net N$13: track 2.54 -> 5.08 mm
- net MOSI: track 9.94 -> 8.67 mm
- net N$2: track 24.5 -> 25.7 mm
- net N$7: track 3.81 -> 2.54 mm
- net N$1: track 25.1 -> 23.8 mm
Other:
- board text added: "GND"
- board text added: "MISO"
- board text added: "MOSI"
- board text added: "PWR"
- board text added: "RST"
- board text added: "SCK"
- board text added: "USB"
- board text added: "USBTiny AVR Programmer v.2.0"
- board text added: "VCC"

Commit message: Version 0.07
Parts:
- moved C1 17.8 mm to (7.62, 29.2), turned to 270 degrees
- moved X1 3.81 mm to (3.81, 16.5)
Routing:
- net GND: track 127.0 -> 135.6 mm
- net N$2: track 25.7 -> 18.9 mm
- net N$1: track 23.8 -> 17.7 mm
- net VCC: track 80.7 -> 84.0 mm
Other:
- board text added: "CC BY-SA 3.0"
- board text added: "PROG"
- board text added: "USBTinyISP AVR Programmer v.2.0"
- board text added: "USB_OK"
- board text added: "github.com/lowvoltage"
- board text added: "www.ladyada.net/make/usbtinyisp"
- board text added: "www.symbolengine.com"
- board text removed: "USBTiny AVR Programmer v.2.0"

Commit message: Version 0.08 - Final tweaks
Parts:
- added U$1: (no value), ohw-logo:OSHW_6X100_NOTEXT
- JP1: value (none) -> ISP_HEADER
- JP3: value PWR -> PWR_JUMPER
- LED1: value (none) -> BURN
- LED2: value (none) -> READY
- X1: value (none) -> USB_CONN
Connections:
- net N$14 renamed VCC_REMOTE
Other:
- board text added: "BURN"
- board text added: "READY"
- board text added: "lowvoltage.wordpress.com"
- board text removed: "PROG"
- board text removed: "USB_OK"
- board text removed: "github.com/lowvoltage"
Changed lines of the file:
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@@
 <wire x1="0" y1="33.02" x2="0" y2="0" width="0" layer="20"/>
 <text x="38.608" y="2.54" size="1.778" layer="16" rot="MR180">USBtinyISP</text>
-<text x="53.975" y="17.145" size="0.8128" layer="25" rot="R45">VCC</text>
-<text x="53.975" y="12.065" size="0.8128" layer="25" rot="R45">GND</text>
-<text x="53.975" y="14.605" size="0.8128" layer="25" rot="R45">MOSI</text>
-<text x="46.99" y="10.16" size="0.8128" layer="25" rot="R45">RST</text>
-<text x="49.53" y="19.685" size="0.8128" layer="25" rot="R45">MISO</text>
-<circle x="48.895" y="19.685" radius="0.254" width="0.4064" layer="25"/>
-<text x="53.34" y="26.67" size="1.016" layer="25">USB</text>
-<text x="53.34" y="25.4" size="1.016" layer="25">PWR</text>
-<text x="12.7" y="30.48" size="1.778" layer="25">USBTinyISP AVR Programmer v.2.0</text>
-<text x="46.99" y="12.7" size="0.8128" layer="25" rot="R45">SCK</text>
-<text x="27.94" y="3.81" size="1.016" layer="25" rot="R90">www.ladyada.net/make/usbtinyisp</text>
-<text x="29.21" y="3.81" size="1.016" layer="25" rot="R90">www.symbolengine.com</text>
-<text x="30.48" y="3.81" size="1.016" layer="25" rot="R90">github.com/lowvoltage</text>
-<text x="41.91" y="12.7" size="1.27" layer="25" rot="R90">CC BY-SA 3.0</text>
-<text x="13.335" y="0.635" size="1.016" layer="25">USB_OK</text>
-<text x="34.29" y="2.54" size="1.016" layer="25">PROG</text>
+<text x="53.975" y="17.145" size="1.016" layer="21" rot="R45">VCC</text>
+<text x="53.975" y="12.065" size="1.016" layer="21" rot="R45">GND</text>
+<text x="53.975" y="14.605" size="1.016" layer="21" rot="R45">MOSI</text>
+<text x="46.355" y="9.525" size="1.016" layer="21" rot="R45">RST</text>
+<text x="49.53" y="19.685" size="1.016" layer="21" rot="R45">MISO</text>
+<circle x="48.895" y="19.685" radius="0.254" width="0.4064" layer="21"/>
+<text x="52.07" y="22.86" size="1.27" layer="21">USB</text>
+<text x="52.07" y="21.59" size="1.27" layer="21">PWR</text>
+<text x="12.7" y="30.48" size="1.778" layer="21">USBTinyISP AVR Programmer v.2.0</text>
+<text x="46.355" y="12.065" size="1.016" layer="21" rot="R45">SCK</text>
+<text x="52.705" y="1.27" size="1.016" layer="21" rot="R180">www.ladyada.net/make/usbtinyisp</text>
+<text x="49.53" y="2.54" size="1.016" layer="21" rot="R180">www.symbolengine.com</text>
+<text x="50.165" y="3.81" size="1.016" layer="21" rot="R180">lowvoltage.wordpress.com</text>
+<text x="28.575" y="20.955" size="1.27" layer="21" rot="R270">CC BY-SA 3.0</text>
+<text x="13.335" y="0.635" size="1.27" layer="21">READY</text>
+<text x="34.29" y="3.81" size="1.27" layer="21">BURN</text>
 </plain>
 <attributes>
@@
 <attribute name="VALUE" x="28.448" y="26.67" size="1.778" layer="27" ratio="10" rot="R270"/>
 </element>
-<element name="JP3" library="pinhead" package="1X02" value="PWR" x="52.07" y="26.67" smashed="yes" rot="R90">
+<element name="JP3" library="pinhead" package="1X02" value="PWR_JUMPER" x="52.07" y="26.67" smashed="yes" rot="R90">
 <attribute name="NAME" x="48.1838" y="29.1338" size="1.27" layer="25" ratio="10" display="off"/>
 <attribute name="VALUE" x="55.245" y="24.13" size="1.27" layer="27" rot="R90"/>
@@
 <attribute name="VALUE" x="4.826" y="31.496" size="1.27" layer="27" ratio="10" rot="R270"/>
 </element>
-<element name="LED1" library="minimidi" package="LED3MM" value="" x="36.83" y="7.62" smashed="yes">
-<attribute name="NAME" x="34.29" y="3.81" size="1.27" layer="25" ratio="10"/>
+<element name="LED1" library="minimidi" package="LED3MM" value="BURN" x="36.83" y="7.62" smashed="yes">
+<attribute name="NAME" x="34.925" y="10.16" size="1.27" layer="25" ratio="10"/>
 <attribute name="VALUE" x="38.735" y="5.969" size="1.27" layer="27" ratio="10"/>
 </element>
@@
 <attribute name="VALUE" x="20.447" y="5.461" size="1.27" layer="27" ratio="10"/>
 </element>
-<element name="LED2" library="minimidi" package="LED3MM" value="" x="20.32" y="3.81" smashed="yes" rot="R270">
+<element name="LED2" library="minimidi" package="LED3MM" value="READY" x="20.32" y="3.81" smashed="yes" rot="R270">
 <attribute name="NAME" x="13.335" y="2.286" size="1.27" layer="25" ratio="10"/>
 <attribute name="VALUE" x="18.669" y="1.905" size="1.27" layer="27" ratio="10" rot="R270"/>
 </element>
-<element name="JP1" library="pinhead-ez" package="2X03" value="" x="50.8" y="15.24" smashed="yes" rot="R270">
+<element name="JP1" library="pinhead-ez" package="2X03" value="ISP_HEADER" x="50.8" y="15.24" smashed="yes" rot="R270">
 <attribute name="NAME" x="50.165" y="17.78" size="1.27" layer="25" ratio="10" rot="R270" display="off"/>
 <attribute name="VALUE" x="46.355" y="19.05" size="1.27" layer="27" rot="R270"/>
 </element>
-<element name="X1" library="con-berg-ez" package="PN61729" value="" x="3.81" y="16.51" smashed="yes" rot="R270">
+<element name="X1" library="con-berg-ez" package="PN61729" value="USB_CONN" x="3.81" y="16.51" smashed="yes" rot="R270">
 <attribute name="NAME" x="2.54" y="16.51" size="1.27" layer="25"/>
 <attribute name="VALUE" x="-5.08" y="8.89" size="1.27" layer="27"/>
@@
 <attribute name="VALUE" x="20.574" y="16.764" size="1.27" layer="27" ratio="10" rot="R90"/>
 </element>
+<element name="U$1" library="ohw-logo" package="OSHW_6X100_NOTEXT" value="" x="23.495" y="0.635"/>
 </elements>
 <signals>
@@
 <wire x1="44.45" y1="12.7" x2="44.45" y2="7.62" width="0.6096" layer="16"/>
 </signal>
-<signal name="N$14">
+<signal name="VCC_REMOTE">
 <contactref element="JP1" pad="2"/>
 <contactref element="JP3" pad="1"/>
