File: USBTinyISP-Single-Sided/usbtiny-v2-SS.sch (EAGLE design)
At the start: 22 parts, among them IC1 ATTINY2313-20P, IC2 74AHC125N, Q1 12Mhz

Commit message: Version 0.03
Parts:
- R2: device rcl-ez:R-US_0207/7 -> rcl-ez:R-US_0207/10
- R3: device rcl-ez:R-US_0207/5V -> rcl-ez:R-US_0207/10
- R5, R6: device rcl-ez:R-US_0207/5V -> rcl-ez:R-US_0207/2V
Changed lines of the file:
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@@
 <parts>
 <part name="R1" library="rcl-ez" deviceset="R-US_" device="0207/10" value="27"/>
-<part name="R2" library="rcl-ez" deviceset="R-US_" device="0207/7" value="27"/>
-<part name="R3" library="rcl-ez" deviceset="R-US_" device="0207/5V" value="1.5K"/>
+<part name="R2" library="rcl-ez" deviceset="R-US_" device="0207/10" value="27"/>
+<part name="R3" library="rcl-ez" deviceset="R-US_" device="0207/10" value="1.5K"/>
 <part name="GND1" library="supply1" deviceset="GND" device=""/>
 <part name="IC1" library="avr" deviceset="ATTINY2313" device="P" technology="-20"/>
@@
 <part name="P+2" library="supply1" deviceset="VCC" device=""/>
 <part name="LED1" library="minimidi" deviceset="LED" device="3MM"/>
-<part name="R6" library="rcl-ez" deviceset="R-US_" device="0207/5V" value="1.5K"/>
+<part name="R6" library="rcl-ez" deviceset="R-US_" device="0207/2V" value="1.5K"/>
 <part name="GND5" library="supply1" deviceset="GND" device=""/>
 <part name="D1" library="diode" deviceset="ZENER-DIODE" device="DO35Z10" value="3.6V"/>
@@
 <part name="R10" library="rcl-ez" deviceset="R-US_" device="0207/10" value="10K"/>
 <part name="P+5" library="supply1" deviceset="VCC" device=""/>
-<part name="R5" library="rcl-ez" deviceset="R-US_" device="0207/5V" value="1.5K"/>
+<part name="R5" library="rcl-ez" deviceset="R-US_" device="0207/2V" value="1.5K"/>
 <part name="LED2" library="minimidi" deviceset="LED" device="3MM"/>
 <part name="JP1" library="pinhead-ez" deviceset="PINHD-2X3" device=""/>
